File: tracer.kicad_pcb (KiCad board)
At the start: 4 copper layers, 22 x 45 mm, 18 parts, among them J1 IO_JACK_F04_SPLIT, K1 Coto-9913-05-20, K2 Coto-9913-05-20, Q1 MMBT3904, Q2 MMBT3904, U1 AD8403ARZ1, U2 AD8403ARZ1

Commit message: Made Project Self-contained
Parts:
- A1: footprint novac:MODULE_TINY_2040 -> .tracer:MODULE_TINY_2040
- A2: footprint novac:MODULE_OLED_490 -> .tracer:MODULE_OLED_490
- D1, D2: footprint novac:DFN1006-2 -> .tracer:DFN1006-2
- J1: footprint novac:SAMTEC-SSQ-102-02-SIDEWAYS -> .tracer:SAMTEC-SSQ-102-02-SIDEWAYS
- K1, K2: footprint novac:REED_RELAY_COTO_9913 -> .tracer:REED_RELAY_COTO_9913
- LOGO1: footprint novac:OSHW-Logo2_7.3x6mm_SilkScreen -> .tracer:OSHW-Logo2_7.3x6mm_SilkScreen
- Q1, Q2: footprint novac:SOT-23 -> .tracer:SOT-23
- R1, R2: footprint novac:R_0805_2012Metric -> .tracer:R_0805_2012Metric
- TP13, TP14, TP17, TP19: footprint novac:via-0.8x0.4 -> .tracer:via-0.8x0.4
- U1, U2: footprint novac:SOIC-24W_7.5x15.4mm_P1.27mm -> .tracer:SOIC-24W_7.5x15.4mm_P1.27mm
