File: tracer.sch (KiCad schematic (older format))
At the start: 18 parts, among them J1 IO_JACK_F04_SPLIT, K1 Coto-9913-05-20, K2 Coto-9913-05-20, Q1 MMBT3904, Q2 MMBT3904, U1 AD8403ARZ1, U2 AD8403ARZ1

Commit message: Made Project Self-contained
Parts:
- A1: footprint novac:MODULE_TINY_2040 -> .tracer:MODULE_TINY_2040; symbol novac:Tiny2040 -> .tracer:Tiny2040
- A2: footprint novac:MODULE_OLED_490 -> .tracer:MODULE_OLED_490; symbol novac:ASSY_OLED_490MILS_62x32_I2C -> .tracer:ASSY_OLED_490MILS_62x32_I2C
- D1, D2: footprint novac:DFN1006-2 -> .tracer:DFN1006-2; symbol novac:DIODE -> .tracer:DIODE
- J1: footprint novac:SAMTEC-SSQ-102-02-SIDEWAYS -> .tracer:SAMTEC-SSQ-102-02-SIDEWAYS; symbol novac:IO_JACK_F04_SPLIT -> .tracer:IO_JACK_F04_SPLIT
- K1, K2: footprint novac:REED_RELAY_COTO_9913 -> .tracer:REED_RELAY_COTO_9913; symbol novac:COTO-9913-REED-RELAY -> .tracer:COTO-9913-REED-RELAY
- LOGO1: footprint novac:OSHW-Logo2_7.3x6mm_SilkScreen -> .tracer:OSHW-Logo2_7.3x6mm_SilkScreen; symbol novac:Logo_Open_Hardware_Small -> .tracer:Logo_Open_Hardware_Small
- Q1, Q2: footprint novac:SOT-23 -> .tracer:SOT-23; symbol novac:MMBT3904 -> .tracer:MMBT3904
- R1, R2: footprint novac:R_0805_2012Metric -> .tracer:R_0805_2012Metric; symbol novac:R_US -> .tracer:R_US
- TP13, TP14, TP17, TP19: footprint novac:via-0.8x0.4 -> .tracer:via-0.8x0.4; symbol novac:TestPoint -> .tracer:TestPoint
- U1, U2: footprint novac:SOIC-24W_7.5x15.4mm_P1.27mm -> .tracer:SOIC-24W_7.5x15.4mm_P1.27mm; symbol novac:AD8403ARZ1 -> .tracer:AD8403ARZ1
Connections:
- net +3V3: now also A2.2 (VCC); no longer A2.3 (VCC)
- net GND: now also A2.1 (GND); no longer A1.18 (GND), A2.4 (GND)
- net at A1.15 (GP1): now also A2.3 (SCL); no longer A2.2 (SCL)
- net at A1.16 (GP0): now also A2.4 (SDA); no longer A2.1 (SDA)
- net at TP17.1: no longer A1.17 (SWC)
- net at TP19.1: no longer A1.19 (SWD)
Changed lines of the file:
@@
 $EndDescr
 $Comp
-L novac:COTO-9913-REED-RELAY K1
+L .tracer:COTO-9913-REED-RELAY K1
 U 1 1 6093F5CC
 P 12400 3700
 F 0 "K1" V 12750 3650 50  0000 L CNN
 F 1 "Coto-9913-05-20" V 12700 3700 50  0001 L CNN
-F 2 "novac:REED_RELAY_COTO_9913" H 12700 3650 50  0001 L CNN
+F 2 ".tracer:REED_RELAY_COTO_9913" H 12700 3650 50  0001 L CNN
 F 3 "" H 12400 3700 50  0001 C CNN
 	1    12400 3700
@@
 $EndComp
 $Comp
-L novac:AD8403ARZ1 U1
+L .tracer:AD8403ARZ1 U1
 U 1 1 609402F4
 P 8500 3700
 F 0 "U1" H 8900 4650 50  0000 L BNN
 F 1 "AD8403ARZ1" H 8450 2700 50  0000 L BNN
-F 2 "novac:SOIC-24W_7.5x15.4mm_P1.27mm" H 8500 3700 50  0001 L BNN
+F 2 ".tracer:SOIC-24W_7.5x15.4mm_P1.27mm" H 8500 3700 50  0001 L BNN
 F 3 "" H 8500 3700 50  0001 L BNN
 	1    8500 3700
@@
 $EndComp
 $Comp
-L novac:Tiny2040 A1
+L .tracer:Tiny2040 A1
 U 1 1 60983233
 P 4300 4750
 F 0 "A1" V 5350 5400 50  0000 C CNN
 F 1 "Tiny2040" H 5150 4000 50  0000 C CNN
-F 2 "novac:MODULE_TINY_2040" H 3875 4550 50  0001 C CNN
+F 2 ".tracer:MODULE_TINY_2040" H 3875 4550 50  0001 C CNN
 F 3 "" H 3875 4550 50  0001 C CNN
 	1    4300 4750
@@
 	7600 2950 7800 2950
 $Comp
-L novac:GND #PWR0101
+L .tracer:GND #PWR0101
 U 1 1 6099CFCF
 P 5500 4900
@@
 	7350 4050 7350 4150
 $Comp
-L novac:GND #PWR0102
+L .tracer:GND #PWR0102
 U 1 1 6099EB4F
 P 7350 4650
@@
 	4650 5850 4650 6000
 $Comp
-L novac:GND #PWR0103
+L .tracer:GND #PWR0103
 U 1 1 609EDA4F
 P 4650 6000
@@
 SIG1A
 $Comp
-L novac:+5V #PWR0105
+L .tracer:+5V #PWR0105
 U 1 1 60AA1EC5
 P 3200 5850
@@
 RELAY2
 $Comp
-L novac:AD8403ARZ1 U2
+L .tracer:AD8403ARZ1 U2
 U 1 1 60AF4B09
 P 8500 5800
 F 0 "U2" H 8900 6750 50  0000 L BNN
 F 1 "AD8403ARZ1" H 8450 4800 50  0000 L BNN
-F 2 "novac:SOIC-24W_7.5x15.4mm_P1.27mm" H 8500 5800 50  0001 L BNN
+F 2 ".tracer:SOIC-24W_7.5x15.4mm_P1.27mm" H 8500 5800 50  0001 L BNN
 F 3 "" H 8500 5800 50  0001 L BNN
 	1    8500 5800
@@
 $EndComp
 $Comp
-L novac:COTO-9913-REED-RELAY K2
+L .tracer:COTO-9913-REED-RELAY K2
 U 1 1 60AF646A
 P 12200 5700
 F 0 "K2" V 12550 5650 50  0000 L CNN
 F 1 "Coto-9913-05-20" V 12500 5700 50  0001 L CNN
-F 2 "novac:REED_RELAY_COTO_9913" H 12500 5650 50  0001 L CNN
+F 2 ".tracer:REED_RELAY_COTO_9913" H 12500 5650 50  0001 L CNN
 F 3 "" H 12200 5700 50  0001 C CNN
 	1    12200 5700
@@
 Connection ~ 10850 5050
 $Comp
-L novac:+5V #PWR0104
+L .tracer:+5V #PWR0104
 U 1 1 60B05569
 P 12400 5150
@@
 	7350 6550 7350 6650
 $Comp
-L novac:GND #PWR0106
+L .tracer:GND #PWR0106
 U 1 1 60BBEE3A
 P 7350 6650
@@
 	6700 3400 7800 3400
 $Comp
-L novac:MMBT3904 Q2
+L .tracer:MMBT3904 Q2
 U 1 1 60AB9105
 P 12300 6650
 F 0 "Q2" H 12500 6725 50  0000 L CNN
 F 1 "MMBT3904" H 12500 6650 50  0000 L CNN
-F 2 "novac:SOT-23" H 12500 6575 50  0001 L CIN
+F 2 ".tracer:SOT-23" H 12500 6575 50  0001 L CIN
 F 3 "https://www.onsemi.com/pub/Collateral/2N3903-D.PDF" H 12300 6650 50  0001 L CNN
 	1    12300 6650
@@
 $EndComp
 $Comp
-L novac:R_US R2
+L .tracer:R_US R2
 U 1 1 60ABAE1C
 P 11750 6950
 F 0 "R2" V 11700 7100 50  0000 C CNN
 F 1 "1K" V 11700 6750 50  0000 C CNN
-F 2 "novac:R_0805_2012Metric" V 11790 6940 50  0001 C CNN
+F 2 ".tracer:R_0805_2012Metric" V 11790 6940 50  0001 C CNN
 F 3 "" H 11750 6950 50  0001 C CNN
 	1    11750 6950
@@
 $EndComp
 $Comp
-L novac:MMBT3904 Q1
+L .tracer:MMBT3904 Q1
 U 1 1 60ADC9F4
 P 12950 7050
 F 0 "Q1" H 13150 7125 50  0000 L CNN
 F 1 "MMBT3904" H 13150 7050 50  0000 L CNN
-F 2 "novac:SOT-23" H 13150 6975 50  0001 L CIN
+F 2 ".tracer:SOT-23" H 13150 6975 50  0001 L CIN
 F 3 "https://www.onsemi.com/pub/Collateral/2N3903-D.PDF" H 12950 7050 50  0001 L CNN
 	1    12950 7050
@@
 	12400 6850 12400 6900
 $Comp
-L novac:GND #PWR0107
+L .tracer:GND #PWR0107
 U 1 1 60AFF091
 P 12400 6900
@@
 	13050 7250 13050 7300
 $Comp
-L novac:GND #PWR0108
+L .tracer:GND #PWR0108
 U 1 1 60AFF6D6
 P 13050 7300
@@
 	12700 7050 12750 7050
 $Comp
-L novac:R_US R1
+L .tracer:R_US R1
 U 1 1 60ADC9FE
 P 12550 7050
 F 0 "R1" V 12600 7200 50  0000 C CNN
 F 1 "1K" V 12600 6850 50  0000 C CNN
-F 2 "novac:R_0805_2012Metric" V 12590 7040 50  0001 C CNN
+F 2 ".tracer:R_0805_2012Metric" V 12590 7040 50  0001 C CNN
 F 3 "" H 12550 7050 50  0001 C CNN
 	1    12550 7050
@@
 $EndComp
 $Comp
-L novac:ASSY_OLED_490MILS_62x32_I2C A2
+L .tracer:ASSY_OLED_490MILS_62x32_I2C A2
 U 1 1 60B700C9
 P 2400 2550
 F 0 "A2" H 2750 2200 79  0000 C CNN
 F 1 "ASSY_OLED_490MILS_62x32_I2C" H 2950 2175 79  0001 C CNN
-F 2 "novac:MODULE_OLED_490" H 2000 3250 79  0001 C CNN
+F 2 ".tracer:MODULE_OLED_490" H 2000 3250 79  0001 C CNN
 F 3 "" H 2000 3250 79  0001 C CNN
 	1    2400 2550
@@
 	4050 5850 4050 6000
 $Comp
-L novac:GND #PWR0109
+L .tracer:GND #PWR0109
 U 1 1 60B7889C
 P 4050 6000
@@
 $EndComp
 $Comp
-L novac:+3V3 #PWR0110
+L .tracer:+3V3 #PWR0110
 U 1 1 60B8E0B1
 P 3000 5850
@@
 	3100 2400 3100 2900
 $Comp
-L novac:GND #PWR0112
+L .tracer:GND #PWR0112
 U 1 1 60C18658
 P 3100 2900
@@
 	5100 4750 5500 4750
 $Comp
-L novac:IO_JACK_F04_SPLIT J1
+L .tracer:IO_JACK_F04_SPLIT J1
 U 1 1 609A8705
 P 11500 3700
 F 0 "J1" H 11450 3900 50  0000 R BNN
 F 1 "IO_JACK_F04_SPLIT" H 11500 3575 50  0001 R TNN
-F 2 "novac:SAMTEC-SSQ-102-02-SIDEWAYS" H 11400 3600 50  0001 C CNN
+F 2 ".tracer:SAMTEC-SSQ-102-02-SIDEWAYS" H 11400 3600 50  0001 C CNN
 F 3 "" H 11400 3600 50  0001 C CNN
 	1    11500 3700
@@
 $EndComp
 $Comp
-L novac:IO_JACK_F04_SPLIT J1
+L .tracer:IO_JACK_F04_SPLIT J1
 U 2 1 609AA4B1
 P 11500 5800
 F 0 "J1" H 11450 6000 50  0000 R BNN
 F 1 "IO_JACK_F04_SPLIT" H 11500 5675 50  0001 R TNN
-F 2 "novac:SAMTEC-SSQ-102-02-SIDEWAYS" H 11400 5700 50  0001 C CNN
+F 2 ".tracer:SAMTEC-SSQ-102-02-SIDEWAYS" H 11400 5700 50  0001 C CNN
 F 3 "" H 11400 5700 50  0001 C CNN
 	2    11500 5800
@@
 $EndComp
 $Comp
-L novac:+3V3 #PWR0111
+L .tracer:+3V3 #PWR0111
 U 1 1 609FE4FA
 P 3500 2300
@@
 $EndComp
 $Comp
-L novac:+3V3 #PWR0113
+L .tracer:+3V3 #PWR0113
 U 1 1 609FEC43
 P 7600 2750
@@
 $EndComp
 $Comp
-L novac:+5V #PWR0114
+L .tracer:+5V #PWR0114
 U 1 1 60A005B2
 P 12600 3050
@@
 	7600 2750 7600 2950
 $Comp
-L novac:+3V3 #PWR0115
+L .tracer:+3V3 #PWR0115
 U 1 1 60A00C09
 P 7600 4850
@@
 	7600 4850 7600 5050
 $Comp
-L novac:DIODE D2
+L .tracer:DIODE D2
 U 1 1 60A62D2E
 P 12850 5700
 F 0 "D2" V 12700 5800 50  0000 C CNN
 F 1 "1N4148W" H 13150 5650 50  0000 C CNN
-F 2 "novac:DFN1006-2" H 12850 5700 50  0001 C CNN
+F 2 ".tracer:DFN1006-2" H 12850 5700 50  0001 C CNN
 F 3 "" H 12850 5700 50  0001 C CNN
 	1    12850 5700
@@
 	12400 6200 12400 6000
 $Comp
-L novac:DIODE D1
+L .tracer:DIODE D1
 U 1 1 60A7F081
 P 13050 3700
 F 0 "D1" V 12900 3800 50  0000 C CNN
 F 1 "1N4148W" H 13350 3650 50  0000 C CNN
-F 2 "novac:DFN1006-2" H 13050 3700 50  0001 C CNN
+F 2 ".tracer:DFN1006-2" H 13050 3700 50  0001 C CNN
 F 3 "" H 13050 3700 50  0001 C CNN
 	1    13050 3700
@@
 	13050 4450 12600 4450
 $Comp
-L novac:TestPoint TP19
+L .tracer:TestPoint TP19
 U 1 1 60A00C06
 P 5200 4650
 F 0 "TP19" V 5200 4920 50  0001 C CNN
 F 1 "TestPoint" H 5200 4850 50  0001 C CNN
-F 2 "novac:via-0.8x0.4" H 5400 4650 50  0001 C CNN
+F 2 ".tracer:via-0.8x0.4" H 5400 4650 50  0001 C CNN
 F 3 "" H 5400 4650 50  0001 C CNN
 	1    5200 4650
@@
 $EndComp
 $Comp
-L novac:TestPoint TP17
+L .tracer:TestPoint TP17
 U 1 1 60A01635
 P 5200 4850
 F 0 "TP17" V 5200 5120 50  0001 C CNN
 F 1 "TestPoint" H 5200 5050 50  0001 C CNN
-F 2 "novac:via-0.8x0.4" H 5400 4850 50  0001 C CNN
+F 2 ".tracer:via-0.8x0.4" H 5400 4850 50  0001 C CNN
 F 3 "" H 5400 4850 50  0001 C CNN
 	1    5200 4850
@@
 	5100 4850 5200 4850
 $Comp
-L novac:TestPoint TP14
+L .tracer:TestPoint TP14
 U 1 1 60A834D5
 P 4150 3300
 F 0 "TP14" V 4150 3570 50  0001 C CNN
 F 1 "TestPoint" H 4150 3500 50  0001 C CNN
-F 2 "novac:via-0.8x0.4" H 4350 3300 50  0001 C CNN
+F 2 ".tracer:via-0.8x0.4" H 4350 3300 50  0001 C CNN
 F 3 "" H 4350 3300 50  0001 C CNN
 	1    4150 3300
@@
 $EndComp
 $Comp
-L novac:TestPoint TP13
+L .tracer:TestPoint TP13
 U 1 1 60A8CF49
 P 4250 3300
 F 0 "TP13" V 4250 3570 50  0001 C CNN
 F 1 "TestPoint" H 4250 3500 50  0001 C CNN
-F 2 "novac:via-0.8x0.4" H 4450 3300 50  0001 C CNN
+F 2 ".tracer:via-0.8x0.4" H 4450 3300 50  0001 C CNN
 F 3 "" H 4450 3300 50  0001 C CNN
 	1    4250 3300
@@
 $EndComp
 $Comp
-L novac:Logo_Open_Hardware_Small LOGO1
+L .tracer:Logo_Open_Hardware_Small LOGO1
 U 1 1 60A81A58
 P 2050 6800
 F 0 "LOGO1" H 2050 7075 50  0001 C CNN
 F 1 "Logo_Open_Hardware_Small" H 2050 6575 50  0001 C CNN
-F 2 "novac:OSHW-Logo2_7.3x6mm_SilkScreen" H 2050 6800 50  0001 C CNN
+F 2 ".tracer:OSHW-Logo2_7.3x6mm_SilkScreen" H 2050 6800 50  0001 C CNN
 F 3 "~" H 2050 6800 50  0001 C CNN
 	1    2050 6800
