File: tracer.sch (KiCad schematic (older format))
At the start: 19 parts, among them J1 IO_JACK_F04_SPLIT, K1 Coto-9913-05-20, K2 Coto-9913-05-20, Q1 MMBT3904, Q2 MMBT3904, U1 AD8403ARZ1, U2 AD8403ARZ1, U3 TXS0101

Commit message: v2 release to PCB shop
Parts:
- removed TP13, TP14, TP17, TP19: TestPoint, .tracer:via-0.8x0.4, symbol .tracer:TestPoint
- added R3, R4: 1K, .tracer:R_0805_2012Metric, symbol .tracer:R_US
- added S1, S2: B3U-3100P-B, .tracer:SW_B3U-3100P-B, symbol .tracer:B3U-3100P-B
- A1: footprint .tracer:MODULE_TINY_2040 -> .tracer:MODULE_TINY_2040_DEV2
- A2: footprint .tracer:MODULE_OLED_490 -> .tracer:MODULE_OLED_490_SMALL_PADS
Connections:
- net +5V: now also R3.2, R4.2
- net GND: now also S1.1, S1.3, S2.1, S2.3
- net SDO1_5V: now also R3.1
- net SDO2: now also R4.1
- net at A1.13 (GP3): now also S1.2
- net at A1.14 (GP2): now also S2.2
Changed lines of the file:
@@
 F 0 "A1" V 4850 5400 50  0000 C CNN
 F 1 "Tiny2040" H 4650 4000 50  0000 C CNN
-F 2 ".tracer:MODULE_TINY_2040" H 3375 4550 50  0001 C CNN
+F 2 ".tracer:MODULE_TINY_2040_DEV2" H 3375 4550 50  0001 C CNN
 F 3 "" H 3375 4550 50  0001 C CNN
 	1    3800 4750
@@
 Wire Wire Line
 	7600 2950 7800 2950
-$Comp
-L .tracer:GND #PWR0101
-U 1 1 6099CFCF
-P 5000 4900
-F 0 "#PWR0101" H 5000 4650 50  0001 C CNN
-F 1 "GND" H 5000 4750 50  0000 C CNN
-F 2 "" H 5000 4900 50  0001 C CNN
-F 3 "" H 5000 4900 50  0001 C CNN
-	1    5000 4900
-	1    0    0    -1
-$EndComp
 Wire Wire Line
 	7800 4050 7350 4050
@@
 	1    0    0    -1
 $EndComp
-Text Label 7000 3400 0    50   ~ 0
+Text Label 7750 3400 2    50   ~ 0
 SDO1_5V
-Text Label 7000 3500 0    50   ~ 0
+Text Label 7750 3500 2    50   ~ 0
 ~SS
-Text Label 7000 3600 0    50   ~ 0
+Text Label 7750 3600 2    50   ~ 0
 CLK
-Text Label 7000 3700 0    50   ~ 0
+Text Label 7750 3700 2    50   ~ 0
 SDO2
-Text Label 7000 3800 0    50   ~ 0
+Text Label 7750 3800 2    50   ~ 0
 ~SHDN
-Text Label 7000 3900 0    50   ~ 0
+Text Label 7750 3900 2    50   ~ 0
 ~RS
 Text Label 7000 6950 0    50   ~ 0
@@
 Wire Wire Line
 	5400 6000 7800 6000
-Text Label 7000 5500 0    50   ~ 0
+Text Label 7750 5500 2    50   ~ 0
 SDO2
-Text Label 7000 5600 0    50   ~ 0
+Text Label 7750 5600 2    50   ~ 0
 ~SS
-Text Label 7000 5700 0    50   ~ 0
+Text Label 7750 5700 2    50   ~ 0
 CLK
-Text Label 7000 5800 0    50   ~ 0
+Text Label 7750 5800 2    50   ~ 0
 SDI
-Text Label 7000 5900 0    50   ~ 0
+Text Label 7750 5900 2    50   ~ 0
 ~SHDN
-Text Label 7000 6000 0    50   ~ 0
+Text Label 7750 6000 2    50   ~ 0
 ~RS
 Wire Wire Line
@@
 	6500 5700 7800 5700
 Wire Wire Line
-	6700 5500 7800 5500
+	6700 5500 7150 5500
 Wire Wire Line
 	5500 5900 7800 5900
@@
 Connection ~ 6600 3500
 Wire Wire Line
-	6700 3400 7800 3400
+	6700 3400 6850 3400
 $Comp
 L .tracer:MMBT3904 Q2
@@
 F 0 "A2" H 2250 2200 79  0000 C CNN
 F 1 "ASSY_OLED_490MILS_62x32_I2C" H 2450 2175 79  0001 C CNN
-F 2 ".tracer:MODULE_OLED_490" H 1500 3250 79  0001 C CNN
+F 2 ".tracer:MODULE_OLED_490_SMALL_PADS" H 1500 3250 79  0001 C CNN
 F 3 "" H 1500 3250 79  0001 C CNN
 	1    1900 2550
@@
 	1    0    0    -1
 $EndComp
-Wire Wire Line
-	5000 4750 5000 4900
-Wire Wire Line
-	4600 4750 5000 4750
 $Comp
 L .tracer:IO_JACK_F04_SPLIT J1
@@
 $EndComp
 Wire Wire Line
-	7600 2750 7600 2950
+	7600 2300 7600 2500
 Wire Wire Line
 	7600 4850 7600 5050
@@
 Wire Wire Line
 	13050 4450 12600 4450
-$Comp
-L .tracer:TestPoint TP19
-U 1 1 60A00C06
-P 4700 4650
-F 0 "TP19" V 4700 4920 50  0001 C CNN
-F 1 "TestPoint" H 4700 4850 50  0001 C CNN
-F 2 ".tracer:via-0.8x0.4" H 4900 4650 50  0001 C CNN
-F 3 "" H 4900 4650 50  0001 C CNN
-	1    4700 4650
-	0    1    1    0
-$EndComp
-$Comp
-L .tracer:TestPoint TP17
-U 1 1 60A01635
-P 4700 4850
-F 0 "TP17" V 4700 5120 50  0001 C CNN
-F 1 "TestPoint" H 4700 5050 50  0001 C CNN
-F 2 ".tracer:via-0.8x0.4" H 4900 4850 50  0001 C CNN
-F 3 "" H 4900 4850 50  0001 C CNN
-	1    4700 4850
-	0    1    1    0
-$EndComp
-Wire Wire Line
-	3650 3300 3650 3650
-Wire Wire Line
-	3750 3650 3750 3300
-Wire Wire Line
-	4600 4650 4700 4650
-Wire Wire Line
-	4600 4850 4700 4850
-$Comp
-L .tracer:TestPoint TP14
-U 1 1 60A834D5
-P 3650 3300
-F 0 "TP14" V 3650 3570 50  0001 C CNN
-F 1 "TestPoint" H 3650 3500 50  0001 C CNN
-F 2 ".tracer:via-0.8x0.4" H 3850 3300 50  0001 C CNN
-F 3 "" H 3850 3300 50  0001 C CNN
-	1    3650 3300
-	1    0    0    -1
-$EndComp
-$Comp
-L .tracer:TestPoint TP13
-U 1 1 60A8CF49
-P 3750 3300
-F 0 "TP13" V 3750 3570 50  0001 C CNN
-F 1 "TestPoint" H 3750 3500 50  0001 C CNN
-F 2 ".tracer:via-0.8x0.4" H 3950 3300 50  0001 C CNN
-F 3 "" H 3950 3300 50  0001 C CNN
-	1    3750 3300
-	1    0    0    -1
-$EndComp
+Wire Wire Line
+	3750 3650 3750 3400
 $Comp
 L .tracer:Logo_Open_Hardware_Small LOGO1
@@
 L .tracer:+5V #PWR0113
 U 1 1 60AD5858
-P 7600 2750
-F 0 "#PWR0113" H 7600 2600 50  0001 C CNN
-F 1 "+5V" H 7600 2890 50  0000 C CNN
-F 2 "" H 7600 2750 50  0001 C CNN
-F 3 "" H 7600 2750 50  0001 C CNN
-	1    7600 2750
+P 7600 2300
+F 0 "#PWR0113" H 7600 2150 50  0001 C CNN
+F 1 "+5V" H 7600 2440 50  0000 C CNN
+F 2 "" H 7600 2300 50  0001 C CNN
+F 3 "" H 7600 2300 50  0001 C CNN
+	1    7600 2300
 	1    0    0    -1
 $EndComp
@@
 	1    0    0    -1
 $EndComp
+$Comp
+L .tracer:R_US R3
+U 1 1 60C5D365
+P 6850 2850
+F 0 "R3" H 6750 3000 50  0000 C CNN
+F 1 "1K" H 6750 2650 50  0000 C CNN
+F 2 ".tracer:R_0805_2012Metric" V 6890 2840 50  0001 C CNN
+F 3 "" H 6850 2850 50  0001 C CNN
+	1    6850 2850
+	-1   0    0    1
+$EndComp
+$Comp
+L .tracer:R_US R4
+U 1 1 60C690E0
+P 7150 2850
+F 0 "R4" H 7050 3000 50  0000 C CNN
+F 1 "1K" H 7050 2650 50  0000 C CNN
+F 2 ".tracer:R_0805_2012Metric" V 7190 2840 50  0001 C CNN
+F 3 "" H 7150 2850 50  0001 C CNN
+	1    7150 2850
+	-1   0    0    1
+$EndComp
+Wire Wire Line
+	6850 3000 6850 3400
+Connection ~ 6850 3400
+Wire Wire Line
+	6850 3400 7800 3400
+Wire Wire Line
+	7150 3000 7150 5500
+Connection ~ 7150 5500
+Wire Wire Line
+	7150 5500 7800 5500
+Wire Wire Line
+	6850 2700 6850 2500
+Wire Wire Line
+	6850 2500 7150 2500
+Connection ~ 7600 2500
+Wire Wire Line
+	7600 2500 7600 2950
+Wire Wire Line
+	7150 2700 7150 2500
+Connection ~ 7150 2500
+Wire Wire Line
+	7150 2500 7600 2500
+$Comp
+L .tracer:B3U-3100P-B S1
+U 1 1 60E5A35A
+P 1950 3500
+F 0 "S1" H 1950 3967 50  0000 C CNN
+F 1 "B3U-3100P-B" H 1950 3876 50  0000 C CNN
+F 2 ".tracer:SW_B3U-3100P-B" H 1950 3500 50  0001 L BNN
+F 3 "" H 1950 3500 50  0001 L BNN
+F 4 "Omron" H 1950 3500 50  0001 L BNN "MANUFACTURER"
+	1    1950 3500
+	-1   0    0    -1
+$EndComp
+$Comp
+L .tracer:B3U-3100P-B S2
+U 1 1 60E5AFAD
+P 1950 4550
+F 0 "S2" H 1950 5017 50  0000 C CNN
+F 1 "B3U-3100P-B" H 1950 4926 50  0000 C CNN
+F 2 ".tracer:SW_B3U-3100P-B" H 1950 4550 50  0001 L BNN
+F 3 "" H 1950 4550 50  0001 L BNN
+F 4 "Omron" H 1950 4550 50  0001 L BNN "MANUFACTURER"
+	1    1950 4550
+	-1   0    0    -1
+$EndComp
+Wire Wire Line
+	1450 3400 1250 3400
+Wire Wire Line
+	1250 3400 1250 4000
+$Comp
+L .tracer:GND #PWR0101
+U 1 1 60E66618
+P 1250 5400
+F 0 "#PWR0101" H 1250 5150 50  0001 C CNN
+F 1 "GND" H 1250 5250 50  0000 C CNN
+F 2 "" H 1250 5400 50  0001 C CNN
+F 3 "" H 1250 5400 50  0001 C CNN
+	1    1250 5400
+	1    0    0    -1
+$EndComp
+Wire Wire Line
+	1950 4950 1950 5050
+Wire Wire Line
+	1950 5050 1250 5050
+Connection ~ 1250 5050
+Wire Wire Line
+	1250 5050 1250 5400
+Wire Wire Line
+	1950 3900 1950 4000
+Wire Wire Line
+	1950 4000 1250 4000
+Connection ~ 1250 4000
+Wire Wire Line
+	1250 4000 1250 4450
+Wire Wire Line
+	2450 4450 2800 4450
+Wire Wire Line
+	2800 4450 2800 3500
+Wire Wire Line
+	2800 3500 3650 3500
+Wire Wire Line
+	3650 3500 3650 3650
+Wire Wire Line
+	2450 3400 3750 3400
+Wire Wire Line
+	1450 4450 1250 4450
+Connection ~ 1250 4450
+Wire Wire Line
+	1250 4450 1250 5050
 $EndSCHEMATC
